File: hw/LED_driver.kicad_pcb (KiCad board)
At the start: 2 copper layers, 72 x 47 mm, 96 parts, among them J1 PROG, J10 ADC_EXT, J11 LED_EN, J2 LED_STRIPS, J3 POWER, J4 SINGLE_POWER, J5 RST, J6 RS485_1, J7 RS485_2, J8 I2C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

Commit message: Prototype version v1.
Routing:
- net GND: track 193.2 -> 190.4 mm, vias 73 -> 68
Other:
- board text added: "RS485 LED driver v1 Jethro 2019"
- board text removed: "RS485 LED driver Jethro 2019"
