File: hw/LED_driver.sch (KiCad schematic (older format))
At the start: 96 parts, among them J1 PROG, J10 ADC_EXT, J11 LED_EN, J2 LED_STRIPS, J3 POWER, J4 SINGLE_POWER, J5 RST, J6 RS485_1, J7 RS485_2, J8 I2C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

Commit message: Prototype version v1.
Parts:
- R23, R4: value 33k -> 33k 1%
- R29: value 1k2 -> 1k5
- R5: value 150k -> 150k 1%
- R6, R7: value 10k -> 10k 1%
Changed lines of the file:
@@
 P 1350 7450
 F 0 "R23" H 1420 7496 50  0000 L CNN
-F 1 "33k" H 1420 7405 50  0000 L CNN
+F 1 "33k 1%" H 1420 7405 50  0000 L CNN
 F 2 "Resistor_SMD:R_0603_1608Metric" V 1280 7450 50  0001 C CNN
 F 3 "" H 1350 7450 50  0001 C CNN
@@
 P 15250 1900
 F 0 "R7" H 15320 1946 50  0000 L CNN
-F 1 "10k" H 15320 1855 50  0000 L CNN
+F 1 "10k 1%" H 15320 1855 50  0000 L CNN
 F 2 "Resistor_SMD:R_0603_1608Metric" V 15180 1900 50  0001 C CNN
 F 3 "" H 15250 1900 50  0001 C CNN
@@
 P 15250 1400
 F 0 "R5" H 15320 1446 50  0000 L CNN
-F 1 "150k" H 15320 1355 50  0000 L CNN
+F 1 "150k 1%" H 15320 1355 50  0000 L CNN
 F 2 "Resistor_SMD:R_0603_1608Metric" V 15180 1400 50  0001 C CNN
 F 3 "" H 15250 1400 50  0001 C CNN
@@
 P 14400 1900
 F 0 "R6" H 14470 1946 50  0000 L CNN
-F 1 "10k" H 14470 1855 50  0000 L CNN
+F 1 "10k 1%" H 14470 1855 50  0000 L CNN
 F 2 "Resistor_SMD:R_0603_1608Metric" V 14330 1900 50  0001 C CNN
 F 3 "" H 14400 1900 50  0001 C CNN
@@
 P 14400 1400
 F 0 "R4" H 14470 1446 50  0000 L CNN
-F 1 "33k" H 14470 1355 50  0000 L CNN
+F 1 "33k 1%" H 14470 1355 50  0000 L CNN
 F 2 "Resistor_SMD:R_0603_1608Metric" V 14330 1400 50  0001 C CNN
 F 3 "" H 14400 1400 50  0001 C CNN
@@
 P 5650 7900
 F 0 "R29" H 5720 7946 50  0000 L CNN
-F 1 "1k2" H 5720 7855 50  0000 L CNN
+F 1 "1k5" H 5720 7855 50  0000 L CNN
 F 2 "Resistor_SMD:R_0603_1608Metric" V 5580 7900 50  0001 C CNN
 F 3 "" H 5650 7900 50  0001 C CNN
