File: hw/LED_driver2/LED_driver2.kicad_pcb (KiCad board)
At the start: 2 copper layers, 60 x 65 mm, 96 parts, among them J1 IO_EN, J2 PROG, J3 SINGLE_POWER, J4 I2C, J5 GPIO, J6 LED_EN, J7 Conn_01x03_Male, J8 RS-485, J9 LED, Q1 Q_PMOS_GSD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

Commit message: Finalization.
Parts:
- added R34: NM, Resistor_SMD:R_0603_1608Metric, F.Cu at (200.4, 50.2)
- added R8: 330R, Resistor_SMD:R_0603_1608Metric, F.Cu at (200.4, 53.3)
- C11, C12, C13: footprint Capacitor_SMD:C_0603_1608Metric -> Resistor_SMD:R_0603_1608Metric
- moved R23 3.69 mm to (197.4, 50.2), turned to 270 degrees
- moved R7 3.10 mm to (198.9, 53.3), turned to 270 degrees
Connections:
- net Net-(F1-Pad1) renamed /A
- net Net-(F2-Pad1) renamed /B
- U4 pad 2: /RS485_RW -> Net-(R34-Pad1)
Routing:
- net /RX: track 3.56 -> 8.60 mm
- net Net-(R34-Pad1): track 0.00 -> 5.00 mm
- net Net-(R7-Pad2): track 34.2 -> 30.1 mm
- net +3V3: track 203.5 -> 200.6 mm
- net /RS485_RW: track 37.2 -> 35.5 mm
- net /TX: track 37.8 -> 36.1 mm
- net GND: vias 31 -> 104
Other:
- outline, holes or cut-outs redrawn
- board text added: "3V3"
- board text added: "GND"
- board text added: "I2C"
- board text added: "IO"
- board text added: "IO0 IO1 IO2 3V3 GND"
- board text added: "IO_EN"
- board text added: "LED driver v2 Jethro 2021"
- board text added: "LED+ LED1- LED+ LED2- LED+ LED3-"
- board text added: "LED_EN"
- board text added: "NRST 3V3 SWDIO SWCLK GND"
- board text added: "RS-485 A B A B"
- board text added: "SCL"
- board text added: "SDA"
- board text added: "SINGLE POWER"
- board text added: "V+ LED (max 48V) +12V GND"
