File: hw/LED_driver2/LED_driver2.sch (KiCad schematic (older format))
At the start: 96 parts, among them J1 IO_EN, J2 PROG, J3 SINGLE_POWER, J4 I2C, J5 GPIO, J6 LED_EN, J7 Conn_01x03_Male, J8 RS-485, J9 LED, Q1 Q_PMOS_GSD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

Commit message: Finalization.
Parts:
- added R34: NM, Resistor_SMD:R_0603_1608Metric, symbol Device:R
- added R8: 330R, Resistor_SMD:R_0603_1608Metric, symbol Device:R
- C1: value C -> 1n; LCSC (none) -> C1588
- C11: footprint Capacitor_SMD:C_0603_1608Metric -> Resistor_SMD:R_0603_1608Metric; LCSC (none) -> C14663
- C12, C13: footprint Capacitor_SMD:C_0603_1608Metric -> Resistor_SMD:R_0603_1608Metric
- C14: LCSC (none) -> C14663
- C15: LCSC (none) -> C57112
- C16: LCSC (none) -> C15849
- C2: value C -> 12p; LCSC (none) -> C38523
- C3: value C -> 12p
- C4, C5: value C -> 1n
- C8: value 10u -> 4u7; LCSC (none) -> C19666
- C9: LCSC (none) -> C59461
- D1: LCSC (none) -> C72043
- F1, F2: value Polyfuse -> nSMD020-16V
- Q10: LCSC (none) -> C8326
- Q4: LCSC (none) -> C2146
- R17: LCSC (none) -> C22843
- R24: LCSC (none) -> C23162
- R31: LCSC (none) -> C22775
- R4: LCSC (none) -> C23352
- R6: LCSC (none) -> C23138
- U2: value M24C02-WMN -> M24C64-WMN; LCSC (none) -> C79988
- U3: LCSC (none) -> C6186
- U4: LCSC (none) -> C8963
Connections:
- net GND: now also R34.2
- net RS485_RW: now also R8.1; no longer U4.2 (~RE~)
- net A: now reaches F1.1, J8.1 (Pin_1), J8.3 (Pin_3)
- net B: now reaches F2.1, J8.2 (Pin_2), J8.4 (Pin_4)
- new net: R34.1, R8.2, U4.2 (~RE~)
Changed lines of the file:
@@
 F 2 "Package_SO:SOIC-8_3.9x4.9mm_P1.27mm" H 10300 9300 50  0001 C CIN
 F 3 "http://www.icbase.com/pdf/SPX/SPX00480106.pdf" H 9250 9650 50  0001 C CNN
+F 4 "C8963" H 9250 9650 50  0001 C CNN "LCSC"
 	1    9250 9650
 	1    0    0    -1
@@
 P 1400 3550
 F 0 "C2" V 1148 3550 50  0000 C CNN
-F 1 "C" V 1239 3550 50  0000 C CNN
+F 1 "12p" V 1239 3550 50  0000 C CNN
 F 2 "Capacitor_SMD:C_0603_1608Metric" H 1438 3400 50  0001 C CNN
 F 3 "~" H 1400 3550 50  0001 C CNN
+F 4 "C38523" V 1400 3550 50  0001 C CNN "LCSC"
 	1    1400 3550
 	0    1    1    0
@@
 P 10100 9550
 F 0 "F1" V 9875 9550 50  0000 C CNN
-F 1 "Polyfuse" V 9966 9550 50  0000 C CNN
+F 1 "nSMD020-16V" V 9966 9550 50  0000 C CNN
 F 2 "Fuse:Fuse_1206_3216Metric" H 10150 9350 50  0001 L CNN
 F 3 "~" H 10100 9550 50  0001 C CNN
@@
 P 10100 9750
 F 0 "F2" V 9875 9750 50  0000 C CNN
-F 1 "Polyfuse" V 9966 9750 50  0000 C CNN
+F 1 "nSMD020-16V" V 9966 9750 50  0000 C CNN
 F 2 "Fuse:Fuse_1206_3216Metric" H 10150 9550 50  0001 L CNN
 F 3 "~" H 10100 9750 50  0001 C CNN
@@
 	1    0    0    -1
 $EndComp
-Wire Wire Line
-	8850 9750 8750 9750
-Wire Wire Line
-	8750 9750 8750 9650
-Wire Wire Line
-	8750 9550 8850 9550
-Wire Wire Line
-	8750 9650 8250 9650
-Connection ~ 8750 9650
-Wire Wire Line
-	8750 9650 8750 9550
-Text Label 8250 9650 0    50   ~ 0
+Text Label 7350 9650 0    50   ~ 0
 RS485_RW
 Wire Wire Line
@@
 F 2 "Capacitor_SMD:C_0603_1608Metric" H 14438 7750 50  0001 C CNN
 F 3 "~" H 14400 7900 50  0001 C CNN
+F 4 "C14663" H 14400 7900 50  0001 C CNN "LCSC"
 	1    14400 7900
 	1    0    0    -1
@@
 F 2 "Resistor_SMD:R_0603_1608Metric" V 13680 1600 50  0001 C CNN
 F 3 "~" H 13750 1600 50  0001 C CNN
+F 4 "C22775" V 13750 1600 50  0001 C CNN "LCSC"
 	1    13750 1600
 	0    1    1    0
@@
 F 2 "Package_TO_SOT_SMD:SOT-23" H 12050 5775 50  0001 L CIN
 F 3 "http://www.unisonic.com.tw/datasheet/S8050.pdf" H 11850 5850 50  0001 L CNN
+F 4 "C2146" H 11850 5850 50  0001 C CNN "LCSC"
 	1    11850 5850
 	1    0    0    -1
@@
 F 2 "Package_TO_SOT_SMD:SOT-23" H 12800 5900 50  0001 C CNN
 F 3 "~" H 12600 5800 50  0001 C CNN
+F 4 "C8326" H 12600 5800 50  0001 C CNN "LCSC"
 	1    12600 5800
 	1    0    0    1
@@
 F 2 "Resistor_SMD:R_0603_1608Metric" V 11380 1900 50  0001 C CNN
 F 3 "~" H 11450 1900 50  0001 C CNN
+F 4 "C23162" V 11450 1900 50  0001 C CNN "LCSC"
 	1    11450 1900
 	0    1    1    0
@@
 P 1400 3850
 F 0 "C3" V 1148 3850 50  0000 C CNN
-F 1 "C" V 1239 3850 50  0000 C CNN
+F 1 "12p" V 1239 3850 50  0000 C CNN
 F 2 "Capacitor_SMD:C_0603_1608Metric" H 1438 3700 50  0001 C CNN
 F 3 "~" H 1400 3850 50  0001 C CNN
@@
 F 2 "Resistor_SMD:R_0603_1608Metric" V 2180 2550 50  0001 C CNN
 F 3 "~" H 2250 2550 50  0001 C CNN
+F 4 "C23352" H 2250 2550 50  0001 C CNN "LCSC"
 	1    2250 2550
 	-1   0    0    1
@@
 F 2 "Resistor_SMD:R_0603_1608Metric" V 3530 2850 50  0001 C CNN
 F 3 "~" H 3600 2850 50  0001 C CNN
+F 4 "C23138" V 3600 2850 50  0001 C CNN "LCSC"
 	1    3600 2850
 	0    1    1    0
@@
 F 2 "LED_SMD:LED_0603_1608Metric" H 5200 6850 50  0001 C CNN
 F 3 "~" H 5200 6850 50  0001 C CNN
+F 4 "C72043" V 5200 6850 50  0001 C CNN "LCSC"
 	1    5200 6850
 	0    -1   -1   0
@@
 P 1250 9450
 F 0 "C1" H 1135 9404 50  0000 R CNN
-F 1 "C" H 1135 9495 50  0000 R CNN
+F 1 "1n" H 1135 9495 50  0000 R CNN
 F 2 "Capacitor_SMD:C_0603_1608Metric" H 1288 9300 50  0001 C CNN
 F 3 "~" H 1250 9450 50  0001 C CNN
+F 4 "C1588" H 1250 9450 50  0001 C CNN "LCSC"
 	1    1250 9450
 	-1   0    0    1
@@
 P 1800 9450
 F 0 "C4" H 1685 9404 50  0000 R CNN
-F 1 "C" H 1685 9495 50  0000 R CNN
+F 1 "1n" H 1685 9495 50  0000 R CNN
 F 2 "Capacitor_SMD:C_0603_1608Metric" H 1838 9300 50  0001 C CNN
 F 3 "~" H 1800 9450 50  0001 C CNN
@@
 P 2250 9450
 F 0 "C5" H 2135 9404 50  0000 R CNN
-F 1 "C" H 2135 9495 50  0000 R CNN
+F 1 "1n" H 2135 9495 50  0000 R CNN
 F 2 "Capacitor_SMD:C_0603_1608Metric" H 2288 9300 50  0001 C CNN
 F 3 "~" H 2250 9450 50  0001 C CNN
@@
 P 5850 4300
 F 0 "U2" H 5850 4781 50  0000 C CNN
-F 1 "M24C02-WMN" H 5850 4690 50  0000 C CNN
+F 1 "M24C64-WMN" H 5850 4690 50  0000 C CNN
 F 2 "Package_SO:SOIC-8_3.9x4.9mm_P1.27mm" H 5850 4650 50  0001 C CNN
 F 3 "http://www.st.com/content/ccc/resource/technical/document/datasheet/b0/d8/50/40/5a/85/49/6f/DM00071904.pdf/files/DM00071904.pdf/jcr:content/translations/en.DM00071904.pdf" H 5900 3800 50  0001 C CNN
+F 4 "C79988" H 5850 4300 50  0001 C CNN "LCSC"
 	1    5850 4300
 	1    0    0    -1
@@
 F 0 "C11" H 13265 1096 50  0000 L CNN
 F 1 "100n" H 13265 1005 50  0000 L CNN
-F 2 "Capacitor_SMD:C_0603_1608Metric" H 13188 900 50  0001 C CNN
+F 2 "Resistor_SMD:R_0603_1608Metric" H 13188 900 50  0001 C CNN
 F 3 "~" H 13150 1050 50  0001 C CNN
+F 4 "C14663" H 13150 1050 50  0001 C CNN "LCSC"
 	1    13150 1050
 	1    0    0    -1
@@
 F 0 "C12" H 13265 3146 50  0000 L CNN
 F 1 "100n" H 13265 3055 50  0000 L CNN
-F 2 "Capacitor_SMD:C_0603_1608Metric" H 13188 2950 50  0001 C CNN
+F 2 "Resistor_SMD:R_0603_1608Metric" H 13188 2950 50  0001 C CNN
 F 3 "~" H 13150 3100 50  0001 C CNN
 	1    13150 3100
@@
 F 0 "C13" H 13265 5146 50  0000 L CNN
 F 1 "100n" H 13265 5055 50  0000 L CNN
-F 2 "Capacitor_SMD:C_0603_1608Metric" H 13188 4950 50  0001 C CNN
+F 2 "Resistor_SMD:R_0603_1608Metric" H 13188 4950 50  0001 C CNN
 F 3 "~" H 13150 5100 50  0001 C CNN
 	1    13150 5100
@@
 F 2 "Resistor_SMD:R_0603_1608Metric" V 6330 3900 50  0001 C CNN
 F 3 "~" H 6400 3900 50  0001 C CNN
+F 4 "C22843" H 6400 3900 50  0001 C CNN "LCSC"
 	1    6400 3900
 	-1   0    0    1
@@
 F 2 "Package_TO_SOT_SMD:SOT-223-3_TabPin2" H 8550 4000 50  0001 C CNN
 F 3 "http://www.advanced-monolithic.com/pdf/ds1117.pdf" H 8650 3550 50  0001 C CNN
+F 4 "C6186" H 8550 3800 50  0001 C CNN "LCSC"
 	1    8550 3800
 	1    0    0    -1
@@
 F 2 "Capacitor_SMD:C_0603_1608Metric" H 9138 3850 50  0001 C CNN
 F 3 "~" H 9100 4000 50  0001 C CNN
+F 4 "C59461" H 9100 4000 50  0001 C CNN "LCSC"
 	1    9100 4000
 	1    0    0    -1
@@
 P 8050 4000
 F 0 "C8" H 8165 4046 50  0000 L CNN
-F 1 "10u" H 8165 3955 50  0000 L CNN
+F 1 "4u7" H 8165 3955 50  0000 L CNN
 F 2 "Capacitor_SMD:C_0603_1608Metric" H 8088 3850 50  0001 C CNN
 F 3 "~" H 8050 4000 50  0001 C CNN
+F 4 "C19666" H 8050 4000 50  0001 C CNN "LCSC"
 	1    8050 4000
 	1    0    0    -1
@@
 F 2 "Capacitor_SMD:C_0603_1608Metric" H 3888 1950 50  0001 C CNN
 F 3 "~" H 3850 2100 50  0001 C CNN
+F 4 "C57112" H 3850 2100 50  0001 C CNN "LCSC"
 	1    3850 2100
 	1    0    0    -1
@@
 F 2 "Capacitor_SMD:C_0603_1608Metric" H 4288 1950 50  0001 C CNN
 F 3 "~" H 4250 2100 50  0001 C CNN
+F 4 "C15849" H 4250 2100 50  0001 C CNN "LCSC"
 	1    4250 2100
 	1    0    0    -1
@@
 Wire Wire Line
 	3400 3250 4250 3250
+$Comp
+L Device:R R8
+U 1 1 608A1C0F
+P 7950 9550
+F 0 "R8" V 7743 9550 50  0000 C CNN
+F 1 "330R" V 7834 9550 50  0000 C CNN
+F 2 "Resistor_SMD:R_0603_1608Metric" V 7880 9550 50  0001 C CNN
+F 3 "~" H 7950 9550 50  0001 C CNN
+	1    7950 9550
+	0    -1   -1   0
+$EndComp
+$Comp
+L Device:R R34
+U 1 1 608A35AD
+P 8150 10050
+F 0 "R34" V 7943 10050 50  0000 C CNN
+F 1 "NM" V 8034 10050 50  0000 C CNN
+F 2 "Resistor_SMD:R_0603_1608Metric" V 8080 10050 50  0001 C CNN
+F 3 "~" H 8150 10050 50  0001 C CNN
+	1    8150 10050
+	1    0    0    -1
+$EndComp
+$Comp
+L power:GND #PWR0172
+U 1 1 608A3D7A
+P 8150 10250
+F 0 "#PWR0172" H 8150 10000 50  0001 C CNN
+F 1 "GND" H 8155 10077 50  0000 C CNN
+F 2 "" H 8150 10250 50  0001 C CNN
+F 3 "" H 8150 10250 50  0001 C CNN
+	1    8150 10250
+	1    0    0    -1
+$EndComp
+Wire Wire Line
+	8150 10250 8150 10200
+Wire Wire Line
+	8150 9900 8150 9550
+Wire Wire Line
+	8150 9550 8100 9550
+Wire Wire Line
+	8150 9550 8850 9550
+Connection ~ 8150 9550
+Wire Wire Line
+	8850 9750 7750 9750
+Wire Wire Line
+	7750 9750 7750 9650
+Wire Wire Line
+	7750 9550 7800 9550
+Wire Wire Line
+	7750 9650 7350 9650
+Connection ~ 7750 9650
+Wire Wire Line
+	7750 9650 7750 9550
+Text Label 10350 9500 0    50   ~ 0
+A
+Text Label 10250 9750 0    50   ~ 0
+B
 $EndSCHEMATC
