File: hw/LED_driver3/LED_driver3.kicad_pcb (KiCad board)
At the start: 2 copper layers, 60 x 60 mm, 129 parts, among them J1 LED_EN, J10 RJ45_Shielded, J2 I2C, J3 PROG, J4 GPIO, J5 POWER, J6 1WIRE1, J7 1WIRE2, J8 LED, J9 RJ45_Shielded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

Commit message: Routed.
Parts:
- removed TP1, TP2, TP3, TP4: TestPoint, TestPoint:TestPoint_THTPad_D2.0mm_Drill1.0mm
- added C41: DNP, Capacitor_SMD:C_0603_1608Metric, F.Cu at (73.3, 130.6)
- added R44: 0, Resistor_SMD:R_0603_1608Metric, F.Cu at (72.5, 129.0)
- J5: footprint Connector_Phoenix_MSTB:PhoenixContact_MSTBA_2,5_2-G-5,08_1x02_P5.08mm_Horizontal -> Connector_Phoenix_MSTB:PhoenixContact_MSTB_2,5_2-GF-5,08_1x02_P5.08mm_Horizontal_ThreadedFlange
- JP1, JP4: moved to B.Cu
- R34: value 0.004R -> 6m
- U5: value INA180 -> INA180A2
- moved C17 186.9 mm to (48.7, 155.5), turned to -90 degrees
- moved C19 185.8 mm to (46.1, 152.4)
- moved C21 185.8 mm to (42.3, 154.9)
- moved C23 185.8 mm to (42.1, 149.9)
- moved C36 185.8 mm to (43.1, 152.4)
- moved L2 185.8 mm to (45.5, 149.4)
- moved R21 185.8 mm to (46.8, 158.2)
- moved R22 185.8 mm to (45.2, 158.2)
- moved R30 185.8 mm to (42.2, 158.2)
- moved R31 185.8 mm to (43.7, 158.2)
- moved U3 185.8 mm to (45.5, 154.9)
- moved C14 185.3 mm to (50.0, 158.5), turned to 180 degrees
- moved JP2 185.3 mm to (54.1, 158.5)
- moved JP3 175.8 mm to (41.8, 143.6), turned to -90 degrees
- moved U4 170.6 mm to (46.9, 137.9), turned to -90 degrees
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Connections:
- C12 pad 1: +3.3V -> +3V3
- C13 pad 1: +3.3V -> +3V3
- C16 pad 1: +3.3V -> +3V3
- C38 pad 2: /LED_COM -> GND
- C39 pad 2: /LED_COM -> GND
- C40 pad 2: /LED_COM -> GND
- R10 pad 1: +3.3V -> +3V3
- U2 pad 1: Net-(U2-PC13) -> unconnected-(U2-PC13-Pad1)
- U2 pad 11: /12V_SENSE -> /VCC_SENSE
- U2 pad 12: /VCC_SENSE -> /12V_SENSE
- U2 pad 17: /O1_SW -> /O3_SW
- U2 pad 19: /O3_SW -> /O1_SW
- U2 pad 36: /SWCLK/BOOT0 -> /SWCLK
- U2 pad 39: Net-(U2-PD1) -> unconnected-(U2-PD1-Pad39)
- U2 pad 4: +3.3V -> +3V3
- U2 pad 41: Net-(U2-PD3) -> unconnected-(U2-PD3-Pad41)
- U2 pad 6: +3.3V -> +3V3
- U5 pad 1: /CUR_SENSE -> Net-(R44-Pad1)
Routing:
- net +3V3: track 0.00 -> 206.0 mm, vias 0 -> 4
- net GND: track 0.00 -> 148.6 mm, vias 0 -> 150
- net +12V: track 0.00 -> 86.5 mm, vias 0 -> 8
- net VCC: track 0.00 -> 72.2 mm, vias 0 -> 1
- net /LED_COM: track 0.00 -> 61.1 mm, vias 0 -> 18
- net Net-(J10-PadSH): track 0.00 -> 59.8 mm
- net /LED2/LED_IN: track 0.00 -> 50.1 mm, vias 0 -> 5
- net /TX: track 0.00 -> 44.1 mm, vias 0 -> 2
- net /RS485_RW: track 0.00 -> 40.8 mm, vias 0 -> 2
- net VCCQ: track 0.00 -> 38.8 mm
- net Net-(R44-Pad1): track 0.00 -> 37.1 mm, vias 0 -> 2
- net Net-(U2-PB11): track 0.00 -> 36.7 mm, vias 0 -> 2
- net Net-(J10-Pad1): track 0.00 -> 23.6 mm
- net /~{RST}: track 0.00 -> 22.2 mm, vias 0 -> 2
- net Net-(J10-Pad3): track 0.00 -> 20.6 mm
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- added copper zone on B.Cu, net GND
- added copper zone on F.Cu, net GND
Other:
- board size 60 x 60 mm -> 50 x 57 mm

Commit message: Silkscreen finished, bugfixes.
Parts:
- added R45: 330R, Resistor_SMD:R_0603_1608Metric, F.Cu at (81.1, 116.1)
- added R46: 330R, Resistor_SMD:R_0603_1608Metric, F.Cu at (78.8, 113.9)
- added R47: 1k5, Resistor_SMD:R_0603_1608Metric, F.Cu at (65.8, 105.2)
- added R48: 1k5, Resistor_SMD:R_0603_1608Metric, F.Cu at (68.9, 105.2)
- moved R12 12.0 mm to (76.1, 111.2), turned to 90 degrees
- moved R11 7.99 mm to (74.2, 111.1), turned to 90 degrees
- moved R29 5.14 mm to (85.4, 123.2)
- moved R28 4.20 mm to (88.5, 126.3)
- moved C28 3.26 mm to (88.1, 130.5), turned to 90 degrees
- moved R27 2.89 mm to (88.0, 117.2)
- moved C9 1.33 mm to (78.9, 105.3), turned to 0 degrees
- moved R26 1.14 mm to (88.1, 121.3), turned to 90 degrees
- moved C7 0.92 mm to (81.9, 105.3), turned to 0 degrees
- moved C3 0.75 mm to (88.0, 105.3), turned to 0 degrees
- moved C4 0.66 mm to (85.0, 105.3), turned to 0 degrees
- moved R14 0.51 mm to (78.0, 111.2)
- moved R20 0.51 mm to (81.0, 111.2)
- moved R6 0.51 mm to (82.5, 111.2)
- moved R8 0.51 mm to (79.5, 111.2)
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Connections:
- J2 pad 3: GND -> +3V3
- J2 pad 4: +3V3 -> GND
- R11 pad 1: /SDA -> /SDA2
- R12 pad 1: /SCL -> /SCL2
- R14 pad 1: Net-(U2-PA8) -> Net-(U2-PA9/NC)
- R18 pad 1: Net-(U2-PB13) -> Net-(U2-PB14)
- R19 pad 1: Net-(U2-PB14) -> Net-(U2-PB15)
- R20 pad 1: Net-(U2-PB15) -> Net-(U2-PA8)
- U1 pad 5: /SDA -> /SDA2
- U1 pad 6: /SCL -> /SCL2
- U2 pad 25: Net-(U2-PB13) -> unconnected-(U2-PB13-Pad25)
- U2 pad 29: unconnected-(U2-PA9/NC-Pad29) -> Net-(U2-PA9/NC)
- U2 pad 30: unconnected-(U2-PC6-Pad30) -> /1WIRE
- U2 pad 33: unconnected-(U2-PA11/PA9-Pad33) -> Net-(U2-PA11/PA9)
- U2 pad 34: unconnected-(U2-PA12/PA10-Pad34) -> Net-(U2-PA12/PA10)
Routing:
- net Net-(U2-PB13): track 20.0 -> 0.00 mm
- net /SCL2: track 0.00 -> 19.9 mm, vias 0 -> 2
- net Net-(U2-PA9/NC): track 0.00 -> 17.3 mm
- net /SDA2: track 0.00 -> 12.3 mm, vias 0 -> 2
- net /1WIRE: track 6.72 -> 18.0 mm, vias 0 -> 2
- net Net-(U2-PA12/PA10): track 0.00 -> 11.0 mm, vias 0 -> 2
- net Net-(U2-PA11/PA9): track 0.00 -> 9.87 mm, vias 0 -> 2
- net /SWDIO: track 16.4 -> 11.9 mm
- net Net-(J7-Pin_2): track 2.60 -> 6.80 mm
- net /SDA: track 9.21 -> 5.06 mm
- net /SCL: track 16.2 -> 12.7 mm
- net Net-(J7-Pin_1): track 2.75 -> 4.89 mm
- net Net-(U2-PB14): track 16.4 -> 18.4 mm
- net Net-(U2-PA8): track 17.5 -> 15.5 mm
- net +3V3: track 206.0 -> 204.1 mm, vias 4 -> 3
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Other:
- board text added: "+VLED"
- board text added: "12V from"
- board text added: "1Wire"
- board text added: "24V to DCDC"
- board text added: "4 - B- 5 - A+ 7 - +12V 8 - GND"
- board text added: "EE WR PROT"
- board text added: "GND"
- board text added: "GND 3V3 IO3/B IO2/A IO1 IO0"
- board text added: "GND 3V3 SCL/TX SDA/RX"
- board text added: "GND DQ 3V3"
- board text added: "GPIO/ENC"
- board text added: "I2C UART"
- board text added: "Jethro, 2024-09-17"
- board text added: "LED EN"
- board text added: "LED1 - +"
- board text added: "LED2 - +"
- board text added: "LED3 - +"
- board text added: "PWM LED Driver"
- board text added: "RJ-45"
- board text added: "RJ-45 DCDC"
- board text added: "RS-485 TERM"
- board text added: "VLED: 9-28V Max 3A per channel"
- board text added: "~{RST} 3V3 SWDIO SWCLK GND"
