File: hw/LED_driver3/driver.kicad_sch (KiCad schematic)
At the start: 7 parts, among them Q1 MDD50N06D, U7 UCC27517DBVR

Commit message: Routed.
Parts:
- renumbered C29 to C32, C27 to C33, C28 to C34, D8 to D9, Q1 to Q3, R40 to R41, U7 to U8
Changed lines of the file:
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@@
 		(dnp no)
 		(fields_autoplaced yes)
-		(property "Reference" "D8"
+		(property "Reference" "D9"
 			(at 184.15 61.9124 90)
 			(effects
@@
 		(dnp no)
 		(fields_autoplaced yes)
-		(property "Reference" "#PWR077"
+		(property "Reference" "#PWR082"
 			(at 149.86 95.25 0)
 			(effects
@@
 		(dnp no)
 		(fields_autoplaced yes)
-		(property "Reference" "#PWR074"
+		(property "Reference" "#PWR084"
 			(at 158.75 62.23 0)
 			(effects
@@
 		(dnp no)
 		(fields_autoplaced yes)
-		(property "Reference" "#PWR073"
+		(property "Reference" "#PWR083"
 			(at 158.75 44.45 0)
 			(effects
@@
 		(dnp no)
 		(fields_autoplaced yes)
-		(property "Reference" "#PWR080"
+		(property "Reference" "#PWR085"
 			(at 181.61 62.23 0)
 			(effects
@@
 		(dnp no)
 		(fields_autoplaced yes)
-		(property "Reference" "C28"
+		(property "Reference" "C34"
 			(at 175.26 46.9899 0)
 			(effects
@@
 		(dnp no)
 		(fields_autoplaced yes)
-		(property "Reference" "C27"
+		(property "Reference" "C33"
 			(at 162.56 46.9899 0)
 			(effects
@@
 		(dnp no)
 		(fields_autoplaced yes)
-		(property "Reference" "C29"
+		(property "Reference" "C32"
 			(at 151.13 46.9899 0)
 			(effects
@@
 		(dnp no)
 		(fields_autoplaced yes)
-		(property "Reference" "Q1"
+		(property "Reference" "Q3"
 			(at 185.42 76.1999 0)
 			(effects
@@
 		(dnp no)
 		(fields_autoplaced yes)
-		(property "Reference" "R40"
+		(property "Reference" "R41"
 			(at 167.64 71.12 90)
 			(effects
@@
 		(on_board yes)
 		(dnp no)
-		(property "Reference" "U7"
+		(property "Reference" "U8"
 			(at 156.464 70.866 0)
 			(effects
@@
 		(dnp no)
 		(fields_autoplaced yes)
-		(property "Reference" "#PWR076"
+		(property "Reference" "#PWR081"
 			(at 149.86 68.58 0)
 			(effects

Commit message: Added LCSC numbers.
Parts:
- Q3: LCSC C99395 -> C5299416
- U8: JLCPCB_CORRECTION (none) -> 0;0;180; LCSC (none) -> C99395
Changed lines of the file:
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@@
 			)
 		)
-		(property "LCSC" "C99395"
+		(property "LCSC" "C5299416"
 			(at 179.07 77.47 0)
 			(effects
@@
 			(at 149.86 77.47 0)
 			(effects
+				(font
+					(size 1.27 1.27)
+				)
+				(hide yes)
+			)
+		)
+		(property "LCSC" "C99395"
+			(at 149.86 77.47 0)
+			(effects
+				(font
+					(size 1.27 1.27)
+				)
+				(hide yes)
+			)
+		)
+		(property "JLCPCB_CORRECTION" "0;0;180"
+			(at 149.86 77.47 0)
+			(effects
